File: v1.1/DSP 1.1.kicad_pcb (KiCad board)
At the start: 2 copper layers, 160.7 x 128.5 mm, 89 parts, among them J1 Conn_01x05_Male, J2 Conn_01x02_Female, P1 EURO_PWR_2x5, Q1 2N3904, U1 TL074, U2 TL072, U3 L7805, U4 PT2399

Commit message: V1.1
Parts:
- added ?: , , F.Cu at (5.72, 186.5)
- added ?: , , F.Cu at (5.64, 214.2)
- added ?: , , F.Cu at (8.69, 243.8)
- added REF**: Mounting Hole, Eurorack:Mounting Hole, F.Cu at (36.7, 139.5)
- added REF**: audio Jack, Eurorack:audio Jack, F.Cu at (18.7, 243.8)
- added REF**: audio Jack, Eurorack:audio Jack, F.Cu at (38.7, 243.8)
- added REF**: Knob, Eurorack:Knob, F.Cu at (32.7, 214.2)
- added REF**: audio Jack, Eurorack:audio Jack, F.Cu at (-0.83, 243.8)
- added REF**: audio Jack, Eurorack:audio Jack, F.Cu at (28.6, 243.8)
- added REF**: Mounting Hole, Eurorack:Mounting Hole, F.Cu at (36.7, 262.0)
- added REF**: Mounting Hole, Eurorack:Mounting Hole, F.Cu at (0.99, 262.0)
- added REF**: Knob, Eurorack:Knob, F.Cu at (34.1, 157.2)
- added REF**: Knob, Eurorack:Knob, F.Cu at (32.7, 186.4)
- added REF**: Mounting Hole, Eurorack:Mounting Hole, F.Cu at (0.99, 139.5)
- added kibuzzard-643BAF55: G***, kibuzzard-643BAF55, F.Cu at (5.57, 198.2)
- added kibuzzard-643BAF55: G***, kibuzzard-643BAF55, F.Cu at (18.9, 251.9)
- added kibuzzard-643BAFC1: G***, kibuzzard-643BAFC1, F.Cu at (8.67, 252.0)
- added kibuzzard-643BAFCE: G***, kibuzzard-643BAFCE, F.Cu at (-0.76, 252.2)
- added kibuzzard-643BAFCE: G***, kibuzzard-643BAFCE, F.Cu at (5.64, 226.3)
- added kibuzzard-643BB32E: G***, kibuzzard-643BB32E, F.Cu at (28.6, 251.8)
- added kibuzzard-643BB339: G***, kibuzzard-643BB339, F.Cu at (38.9, 251.8)
- added kibuzzard-643BB390: G***, kibuzzard-643BB390, F.Cu at (32.7, 198.3)
- added kibuzzard-643BB3B1: G***, kibuzzard-643BB3B1, F.Cu at (33.0, 226.0)
- added kibuzzard-644033EB: G***, kibuzzard-644033EB, F.Cu at (18.4, 258.8)
- added kibuzzard-644033FD: G***, kibuzzard-644033FD, F.Cu at (22.7, 262.3)
- added kibuzzard-64D80CCD: G***, kibuzzard-64D80CCD, F.Cu at (19.6, 139.4)
Other:
- board size 160.7 x 128.5 mm -> 161.3 x 263.9 mm
- board text added: "Alumium Front Panel"
- board text added: "FR4 Front Panel"
- board text added: "Interface / Clock modulator Board"
- board text added: "Main Board"
